Commit message: fixed urdf

File: ros2_ws/src/robot_description/urdf/two_wheel_robot.urdf.xacro (robot description, xacro)
@@ -6,4 +6,5 @@
     <xacro:include filename="$(find robot_description)/urdf/two_wheel_robot_ros2_control.urdf.xacro" />
     <!-- Links -->
+    <link name="base_footprint"/>
     <link name="base_link">
         <inertial>
@@ -85,4 +86,9 @@
     </link>
     <!-- Joints -->
+    <joint name="base_footprint_joint" type="fixed">
+        <parent link="base_footprint"/>
+        <child link="base_link"/>
+        <origin xyz="0 0 0.05" rpy="0 0 0"/>
+    </joint>
     <joint name="left_wheel_joint" type="continuous">
         <parent link="base_link"/>

Commit message: fixed orientation

File: ros2_ws/src/robot_description/urdf/two_wheel_robot.urdf.xacro (robot description, xacro)
@@ -22,5 +22,5 @@
             <origin xyz="0 0 0.1"/>
             <geometry>
-                <box size="0.4 0.2 0.2"/>
+                <box size="0.2 0.4 0.2"/>
             </geometry>
             <material name="blue">
@@ -31,5 +31,5 @@
             <origin xyz="0 0 0.1"/>
             <geometry>
-                <box size="0.4 0.2 0.2"/>
+                <box size="0.2 0.4 0.2"/>
             </geometry>
         </collision>
@@ -45,5 +45,5 @@
         </inertial>
         <visual>
-            <origin xyz="0 0 0" rpy="0 1.5707 0"/>
+            <origin xyz="0 0 0" rpy="1.5707 0 0"/>
             <geometry>
                 <cylinder radius="0.05" length="0.03"/>
@@ -54,5 +54,5 @@
         </visual>
         <collision>
-            <origin xyz="0 0 0" rpy="0 1.5707 0"/>
+            <origin xyz="0 0 0" rpy="1.5707 0 0"/>
             <geometry>
                 <cylinder radius="0.05" length="0.03"/>
@@ -70,5 +70,5 @@
         </inertial>
         <visual>
-            <origin xyz="0 0 0" rpy="0 1.5707 0"/>
+            <origin xyz="0 0 0" rpy="1.5707 0 0"/>
             <geometry>
                 <cylinder radius="0.05" length="0.03"/>
@@ -79,5 +79,5 @@
         </visual>
         <collision>
-            <origin xyz="0 0 0" rpy="0 1.5707 0"/>
+            <origin xyz="0 0 0" rpy="1.5707 0 0"/>
             <geometry>
                 <cylinder radius="0.05" length="0.03"/>
@@ -94,6 +94,6 @@
         <parent link="base_link"/>
         <child link="left_wheel"/>
-        <origin xyz="0.215 0 0"/>
-        <axis xyz="1 0 0"/>
+        <origin xyz="0 0.215 0"/>
+        <axis xyz="0 1 0"/>
         <dynamics damping="0.1" friction="0.1"/>
     </joint>
@@ -101,6 +101,6 @@
         <parent link="base_link"/>
         <child link="right_wheel"/>
-        <origin xyz="-0.215 0 0"/>
-        <axis xyz="1 0 0"/>
+        <origin xyz="0 -0.215 0"/>
+        <axis xyz="0 1 0"/>
         <dynamics damping="0.1" friction="0.1"/>
     </joint>

Commit message: updated physics

File: ros2_ws/src/robot_description/urdf/two_wheel_robot.urdf.xacro (robot description, xacro)
@@ -9,13 +9,13 @@
     <link name="base_link">
         <inertial>
-            <origin xyz="0 0 0"/>
-            <mass value="5.0"/>
+            <origin xyz="0 0 0.03"/>
+            <mass value="3.0"/>
             <inertia
-                ixx="0.2"
+                ixx="0.05"
                 ixy="0.0"
                 ixz="0.0"
-                iyy="0.2"
+                iyy="0.05"
                 iyz="0.0"
-                izz="0.2"/>
+                izz="0.1"/>
         </inertial>
         <visual>
@@ -38,14 +38,14 @@
         <inertial>
             <origin xyz="0 0 0"/>
-            <mass value="0.3"/>
+            <mass value="0.5"/>
             <inertia
-                ixx="0.0005" ixy="0.0" ixz="0.0"
-                iyy="0.0005" iyz="0.0"
-                izz="0.0005"/>
+                ixx="0.0015" ixy="0.0" ixz="0.0"
+                iyy="0.0025" iyz="0.0"
+                izz="0.0015"/>
         </inertial>
         <visual>
             <origin xyz="0 0 0" rpy="1.5707 0 0"/>
             <geometry>
-                <cylinder radius="0.05" length="0.03"/>
+                <cylinder radius="0.08" length="0.03"/>
             </geometry>
             <material name="black">
@@ -56,5 +56,5 @@
             <origin xyz="0 0 0" rpy="1.5707 0 0"/>
             <geometry>
-                <cylinder radius="0.05" length="0.03"/>
+                <cylinder radius="0.08" length="0.03"/>
             </geometry>
         </collision>
@@ -63,14 +63,14 @@
         <inertial>
             <origin xyz="0 0 0"/>
-            <mass value="0.3"/>
+            <mass value="0.5"/>
             <inertia
-                ixx="0.0005" ixy="0.0" ixz="0.0"
-                iyy="0.0005" iyz="0.0"
-                izz="0.0005"/>
+                ixx="0.0015" ixy="0.0" ixz="0.0"
+                iyy="0.0025" iyz="0.0"
+                izz="0.0015"/>
         </inertial>
         <visual>
             <origin xyz="0 0 0" rpy="1.5707 0 0"/>
             <geometry>
-                <cylinder radius="0.05" length="0.03"/>
+                <cylinder radius="0.08" length="0.03"/>
             </geometry>
             <material name="black">
@@ -81,5 +81,5 @@
             <origin xyz="0 0 0" rpy="1.5707 0 0"/>
             <geometry>
-                <cylinder radius="0.05" length="0.03"/>
+                <cylinder radius="0.08" length="0.03"/>
             </geometry>
         </collision>
@@ -89,5 +89,5 @@
         <parent link="base_footprint"/>
         <child link="base_link"/>
-        <origin xyz="0 0 0.05" rpy="0 0 0"/>
+        <origin xyz="0 0 0.08" rpy="0 0 0"/>
     </joint>
     <joint name="left_wheel_joint" type="continuous">
@@ -96,5 +96,5 @@
         <origin xyz="0 0.215 0"/>
         <axis xyz="0 1 0"/>
-        <dynamics damping="0.1" friction="0.1"/>
+        <dynamics damping="0.0" friction="0.0"/>
     </joint>
     <joint name="right_wheel_joint" type="continuous">
@@ -103,5 +103,5 @@
         <origin xyz="0 -0.215 0"/>
         <axis xyz="0 1 0"/>
-        <dynamics damping="0.1" friction="0.1"/>
+        <dynamics damping="0.0" friction="0.0"/>
     </joint>
     <!-- IMU -->

File: ros2_ws/src/robot_description/urdf/two_wheel_robot_gazebo.urdf.xacro (robot description, xacro)
@@ -2,15 +2,15 @@
 <robot name="two_wheel_robot" xmlns:xacro="http://www.ros.org/wiki/xacro">
     <gazebo reference="left_wheel">
-        <mu1>3.0</mu1>
-        <mu2>3.0</mu2>
+        <mu1>1.0</mu1>
+        <mu2>1.0</mu2>
     </gazebo>
     <gazebo reference="right_wheel">
-        <mu1>3.0</mu1>
-        <mu2>3.0</mu2>
+        <mu1>1.0</mu1>
+        <mu2>1.0</mu2>
     </gazebo>
     <gazebo reference="imu_link">
         <sensor name="imu_sensor" type="imu">
             <always_on>true</always_on>
-            <update_rate>100</update_rate>
+            <update_rate>500</update_rate>
             <visualize>true</visualize>
             <topic>imu</topic>

Commit message: added dynamics

File: ros2_ws/src/robot_description/urdf/two_wheel_robot.urdf.xacro (robot description, xacro)
@@ -96,5 +96,5 @@
         <origin xyz="0 0.215 0"/>
         <axis xyz="0 1 0"/>
-        <dynamics damping="0.0" friction="0.0"/>
+        <dynamics damping="0.01" friction="0.01"/>
     </joint>
     <joint name="right_wheel_joint" type="continuous">
@@ -103,5 +103,5 @@
         <origin xyz="0 -0.215 0"/>
         <axis xyz="0 1 0"/>
-        <dynamics damping="0.0" friction="0.0"/>
+        <dynamics damping="0.01" friction="0.01"/>
     </joint>
     <!-- IMU -->

Commit message: updated robot body

File: ros2_ws/src/robot_description/urdf/two_wheel_robot.urdf.xacro (robot description, xacro)
@@ -19,17 +19,60 @@
                 izz="0.1"/>
         </inertial>
+        <!-- Lower plate -->
         <visual>
-            <origin xyz="0 0 0.1"/>
+            <origin xyz="0 0 0.045"/>
             <geometry>
-                <box size="0.2 0.4 0.2"/>
+                <box size="0.22 0.30 0.005"/>
             </geometry>
-            <material name="blue">
-                <color rgba="0 0 1 1"/>
+            <material name="black">
+                <color rgba="0.1 0.1 0.1 1"/>
             </material>
         </visual>
+        <!-- Upper plate -->
+        <visual>
+            <origin xyz="0 0 0.145"/>
+            <geometry>
+                <box size="0.22 0.30 0.005"/>
+            </geometry>
+            <material name="black"/>
+        </visual>
+        <!-- Front left standoff -->
+        <visual>
+            <origin xyz="0.09 0.12 0.095"/>
+            <geometry>
+                <cylinder radius="0.005" length="0.10"/>
+            </geometry>
+            <material name="gold">
+                <color rgba="0.85 0.70 0.20 1"/>
+            </material>
+        </visual>
+        <!-- Front right standoff -->
+        <visual>
+            <origin xyz="0.09 -0.12 0.095"/>
+            <geometry>
+                <cylinder radius="0.005" length="0.10"/>
+            </geometry>
+            <material name="gold"/>
+        </visual>
+        <!-- Rear left standoff -->
+        <visual>
+            <origin xyz="-0.09 0.12 0.095"/>
+            <geometry>
+                <cylinder radius="0.005" length="0.10"/>
+            </geometry>
+            <material name="gold"/>
+        </visual>
+        <!-- Rear right standoff -->
+        <visual>
+            <origin xyz="-0.09 -0.12 0.095"/>
+            <geometry>
+                <cylinder radius="0.005" length="0.10"/>
+            </geometry>
+            <material name="gold"/>
+        </visual>
         <collision>
-            <origin xyz="0 0 0.1"/>
+            <origin xyz="0 0 0.095"/>
             <geometry>
-                <box size="0.2 0.4 0.2"/>
+                <box size="0.22 0.30 0.11"/>
             </geometry>
         </collision>

Commit message: updated inertial values

File: ros2_ws/src/robot_description/urdf/two_wheel_robot.urdf.xacro (robot description, xacro)
@@ -9,13 +9,13 @@
     <link name="base_link">
         <inertial>
-            <origin xyz="0 0 0.03"/>
-            <mass value="3.0"/>
+            <origin xyz="0 0 0.095"/>
+            <mass value="0.80"/>
             <inertia
-                ixx="0.05"
+                ixx="0.00681"
                 ixy="0.0"
                 ixz="0.0"
-                iyy="0.05"
+                iyy="0.00404"
                 iyz="0.0"
-                izz="0.1"/>
+                izz="0.00923"/>
         </inertial>
         <!-- Lower plate -->
